File: Kicad_project/Placa_seguidor/Placa.sch (KiCad schematic (older format))
At the start: 15 parts, among them J1 Conn_01x02_Female, J2 Conn_01x08_Female, U1 barra2pins, U10 PW_Slinha, U13 Desenho_placa_seguidor, U2 barra3pins, U3 Borne, U4 Borne, U5 Borne, U6 Borne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

Commit message: Implemented another control rules
Parts:
- added C1, C2, C3, C4, C5, C6: C, Capacitor_THT:C_Disc_D5.1mm_W3.2mm_P5.00mm, symbol pspice:C
- added J3: Conn_01x06_Female, Connector_PinSocket_2.54mm:PinSocket_1x06_P2.54mm_Vertical, symbol Connector:Conn_01x06_Female
- added Reg_5V1: LM7805, Package_TO_SOT_THT:TO-220-3_Vertical, symbol Regulator_Linear:LM7805_TO220
Connections:
- net GND: now also C1.1, C2.1, C3.1, C4.1, C5.1, C6.1, J3.4 (Pin_4), Reg_5V1.2 (GND)
- net V3.3: now also C1.2, C3.2, C4.2, C5.2, C6.2
- net VCC: now also Reg_5V1.1 (VI)
- net RX_module: now reaches U8.35 (B10)
- net RX_module: now also J3.2 (Pin_2)
- net TX_module: now reaches U8.36 (B11)
- net TX_module: now also J3.3 (Pin_3)
- new net EN: J3.6 (Pin_6)
- new net State: J3.1 (Pin_1)
- new net V5: C2.2, J3.5 (Pin_5), Reg_5V1.3 (VO)
Changed lines of the file:
@@
 EESchema Schematic File Version 4
 LIBS:Placa-cache
-EELAYER 26 0
+EELAYER 29 0
 EELAYER END
 $Descr A4 11693 8268
@@
 	1    0    0    -1
 $EndComp
+$Comp
+L Regulator_Linear:LM7805_TO220 Reg_5V1
+U 1 1 5D2217A8
+P 3500 3500
+F 0 "Reg_5V1" H 3500 3742 50  0000 C CNN
+F 1 "LM7805" H 3500 3651 50  0000 C CNN
+F 2 "Package_TO_SOT_THT:TO-220-3_Vertical" H 3500 3725 50  0001 C CIN
+F 3 "http://www.fairchildsemi.com/ds/LM/LM7805.pdf" H 3500 3450 50  0001 C CNN
+	1    3500 3500
+	1    0    0    -1
+$EndComp
+Text Label 3200 3500 2    60   ~ 0
+VCC
+Text Label 3500 3800 2    60   ~ 0
+GND
+Text Label 3800 3500 0    60   ~ 0
+V5
+$Comp
+L Connector:Conn_01x06_Female J3
+U 1 1 5D2239CA
+P 4800 3500
+F 0 "J3" H 4828 3476 50  0000 L CNN
+F 1 "Conn_01x06_Female" H 4828 3385 50  0000 L CNN
+F 2 "Connector_PinSocket_2.54mm:PinSocket_1x06_P2.54mm_Vertical" H 4800 3500 50  0001 C CNN
+F 3 "~" H 4800 3500 50  0001 C CNN
+	1    4800 3500
+	1    0    0    -1
+$EndComp
+Text Label 4600 3300 2    60   ~ 0
+State
+Text Label 4600 3400 2    60   ~ 0
+RX_module
+Text Label 4600 3500 2    60   ~ 0
+TX_module
+Text Label 4600 3600 2    60   ~ 0
+GND
+Text Label 4600 3700 2    60   ~ 0
+V5
+Text Label 4600 3800 2    60   ~ 0
+EN
+Text Label 5150 4750 0    60   ~ 0
+RX_module
+Text Label 5150 4650 0    60   ~ 0
+TX_module
+$Comp
+L pspice:C C3
+U 1 1 5D229281
+P 7400 3400
+F 0 "C3" H 7222 3354 50  0000 R CNN
+F 1 "C" H 7222 3445 50  0000 R CNN
+F 2 "Capacitor_THT:C_Disc_D5.1mm_W3.2mm_P5.00mm" H 7400 3400 50  0001 C CNN
+F 3 "~" H 7400 3400 50  0001 C CNN
+	1    7400 3400
+	-1   0    0    1
+$EndComp
+$Comp
+L pspice:C C2
+U 1 1 5D22A0EF
+P 6850 3400
+F 0 "C2" H 6672 3354 50  0000 R CNN
+F 1 "C" H 6672 3445 50  0000 R CNN
+F 2 "Capacitor_THT:C_Disc_D5.1mm_W3.2mm_P5.00mm" H 6850 3400 50  0001 C CNN
+F 3 "~" H 6850 3400 50  0001 C CNN
+	1    6850 3400
+	-1   0    0    1
+$EndComp
+$Comp
+L pspice:C C1
+U 1 1 5D22D2F6
+P 6450 3400
+F 0 "C1" H 6272 3354 50  0000 R CNN
+F 1 "C" H 6272 3445 50  0000 R CNN
+F 2 "Capacitor_THT:C_Disc_D5.1mm_W3.2mm_P5.00mm" H 6450 3400 50  0001 C CNN
+F 3 "~" H 6450 3400 50  0001 C CNN
+	1    6450 3400
+	-1   0    0    1
+$EndComp
+Text Label 6450 3150 0    60   ~ 0
+V3.3
+Text Label 6850 3150 2    60   ~ 0
+V5
+Text Label 7400 3150 2    60   ~ 0
+V3.3
+Text Label 6450 3650 2    60   ~ 0
+GND
+Text Label 6850 3650 2    60   ~ 0
+GND
+Text Label 7400 3650 2    60   ~ 0
+GND
+$Comp
+L pspice:C C4
+U 1 1 5D24620B
+P 7950 3400
+F 0 "C4" H 7772 3354 50  0000 R CNN
+F 1 "C" H 7772 3445 50  0000 R CNN
+F 2 "Capacitor_THT:C_Disc_D5.1mm_W3.2mm_P5.00mm" H 7950 3400 50  0001 C CNN
+F 3 "~" H 7950 3400 50  0001 C CNN
+	1    7950 3400
+	-1   0    0    1
+$EndComp
+Text Label 7950 3150 2    60   ~ 0
+V3.3
+Text Label 7950 3650 2    60   ~ 0
+GND
+$Comp
+L pspice:C C5
+U 1 1 5D247080
+P 8500 3400
+F 0 "C5" H 8322 3354 50  0000 R CNN
+F 1 "C" H 8322 3445 50  0000 R CNN
+F 2 "Capacitor_THT:C_Disc_D5.1mm_W3.2mm_P5.00mm" H 8500 3400 50  0001 C CNN
+F 3 "~" H 8500 3400 50  0001 C CNN
+	1    8500 3400
+	-1   0    0    1
+$EndComp
+Text Label 8500 3150 2    60   ~ 0
+V3.3
+Text Label 8500 3650 2    60   ~ 0
+GND
+$Comp
+L pspice:C C6
+U 1 1 5D24A4F0
+P 9100 3400
+F 0 "C6" H 8922 3354 50  0000 R CNN
+F 1 "C" H 8922 3445 50  0000 R CNN
+F 2 "Capacitor_THT:C_Disc_D5.1mm_W3.2mm_P5.00mm" H 9100 3400 50  0001 C CNN
+F 3 "~" H 9100 3400 50  0001 C CNN
+	1    9100 3400
+	-1   0    0    1
+$EndComp
+Text Label 9100 3150 2    60   ~ 0
+V3.3
+Text Label 9100 3650 2    60   ~ 0
+GND
 $EndSCHEMATC

Commit message: it seems to be working now
Parts:
- removed C1, C2, C3, C4, C5, C6: C, Capacitor_THT:C_Disc_D5.1mm_W3.2mm_P5.00mm, symbol pspice:C
- removed U2: barra3pins, FootLibAlan:barra3pins, symbol Placa-rescue:barra3pins
- added F1: Fuse_Small, Resistor_THT:R_Axial_DIN0309_L9.0mm_D3.2mm_P5.08mm_Vertical, symbol Device:Fuse_Small
- added U2: barra2pins, FootLibAlan:barra2pins, symbol Placa-rescue:barra2pins
Connections:
- net VBat: now also F1.1
- net VCC: now also U2.2 (b)
- new net Vfuse: F1.2, U2.1 (a)
Changed lines of the file:
@@
-$EndComp
-$Comp
-L Placa-rescue:barra3pins U2
-U 1 1 5B006A71
-P 1650 3350
-F 0 "U2" H 1850 3350 60  0000 C CNN
-F 1 "barra3pins" H 1650 3500 60  0000 C CNN
-F 2 "FootLibAlan:barra3pins" H 1650 3350 60  0001 C CNN
-F 3 "" H 1650 3350 60  0001 C CNN
-	1    1650 3350
-	1    0    0    -1
 $EndComp
 $Comp
@@
 Text Label 1100 3600 0    60   ~ 0
 VBat
-Text Label 1650 3600 3    60   ~ 0
-VCC
-Text Label 1550 3600 3    60   ~ 0
+Text Label 1800 3550 3    60   ~ 0
+VCC
+Text Label 1300 2950 2    60   ~ 0
 VBat
 Text Label 1000 3600 2    60   ~ 0
@@
 TX_module
 $Comp
-L pspice:C C3
-U 1 1 5D229281
-P 7400 3400
-F 0 "C3" H 7222 3354 50  0000 R CNN
-F 1 "C" H 7222 3445 50  0000 R CNN
-F 2 "Capacitor_THT:C_Disc_D5.1mm_W3.2mm_P5.00mm" H 7400 3400 50  0001 C CNN
-F 3 "~" H 7400 3400 50  0001 C CNN
-	1    7400 3400
-	-1   0    0    1
-$EndComp
-$Comp
-L pspice:C C2
-U 1 1 5D22A0EF
-P 6850 3400
-F 0 "C2" H 6672 3354 50  0000 R CNN
-F 1 "C" H 6672 3445 50  0000 R CNN
-F 2 "Capacitor_THT:C_Disc_D5.1mm_W3.2mm_P5.00mm" H 6850 3400 50  0001 C CNN
-F 3 "~" H 6850 3400 50  0001 C CNN
-	1    6850 3400
-	-1   0    0    1
-$EndComp
-$Comp
-L pspice:C C1
-U 1 1 5D22D2F6
-P 6450 3400
-F 0 "C1" H 6272 3354 50  0000 R CNN
-F 1 "C" H 6272 3445 50  0000 R CNN
-F 2 "Capacitor_THT:C_Disc_D5.1mm_W3.2mm_P5.00mm" H 6450 3400 50  0001 C CNN
-F 3 "~" H 6450 3400 50  0001 C CNN
-	1    6450 3400
-	-1   0    0    1
-$EndComp
-Text Label 6450 3150 0    60   ~ 0
-V3.3
-Text Label 6850 3150 2    60   ~ 0
-V5
-Text Label 7400 3150 2    60   ~ 0
-V3.3
-Text Label 6450 3650 2    60   ~ 0
-GND
-Text Label 6850 3650 2    60   ~ 0
-GND
-Text Label 7400 3650 2    60   ~ 0
-GND
-$Comp
-L pspice:C C4
-U 1 1 5D24620B
-P 7950 3400
-F 0 "C4" H 7772 3354 50  0000 R CNN
-F 1 "C" H 7772 3445 50  0000 R CNN
-F 2 "Capacitor_THT:C_Disc_D5.1mm_W3.2mm_P5.00mm" H 7950 3400 50  0001 C CNN
-F 3 "~" H 7950 3400 50  0001 C CNN
-	1    7950 3400
-	-1   0    0    1
-$EndComp
-Text Label 7950 3150 2    60   ~ 0
-V3.3
-Text Label 7950 3650 2    60   ~ 0
-GND
-$Comp
-L pspice:C C5
-U 1 1 5D247080
-P 8500 3400
-F 0 "C5" H 8322 3354 50  0000 R CNN
-F 1 "C" H 8322 3445 50  0000 R CNN
-F 2 "Capacitor_THT:C_Disc_D5.1mm_W3.2mm_P5.00mm" H 8500 3400 50  0001 C CNN
-F 3 "~" H 8500 3400 50  0001 C CNN
-	1    8500 3400
-	-1   0    0    1
-$EndComp
-Text Label 8500 3150 2    60   ~ 0
-V3.3
-Text Label 8500 3650 2    60   ~ 0
-GND
-$Comp
-L pspice:C C6
-U 1 1 5D24A4F0
-P 9100 3400
-F 0 "C6" H 8922 3354 50  0000 R CNN
-F 1 "C" H 8922 3445 50  0000 R CNN
-F 2 "Capacitor_THT:C_Disc_D5.1mm_W3.2mm_P5.00mm" H 9100 3400 50  0001 C CNN
-F 3 "~" H 9100 3400 50  0001 C CNN
-	1    9100 3400
-	-1   0    0    1
-$EndComp
-Text Label 9100 3150 2    60   ~ 0
-V3.3
-Text Label 9100 3650 2    60   ~ 0
-GND
+L Placa-rescue:barra2pins U2
+U 1 1 5D66E07C
+P 1850 3300
+F 0 "U2" H 1900 3300 60  0000 C CNN
+F 1 "barra2pins" H 1750 3450 60  0000 C CNN
+F 2 "FootLibAlan:barra2pins" H 1850 3300 60  0001 C CNN
+F 3 "" H 1850 3300 60  0001 C CNN
+	1    1850 3300
+	1    0    0    -1
+$EndComp
+$Comp
+L Device:Fuse_Small F1
+U 1 1 5D67C310
+P 1400 2950
+F 0 "F1" H 1400 3135 50  0000 C CNN
+F 1 "Fuse_Small" H 1400 3044 50  0000 C CNN
+F 2 "Resistor_THT:R_Axial_DIN0309_L9.0mm_D3.2mm_P5.08mm_Vertical" H 1400 2950 50  0001 C CNN
+F 3 "~" H 1400 2950 50  0001 C CNN
+	1    1400 2950
+	1    0    0    -1
+$EndComp
+Text Label 1500 2950 0    50   ~ 0
+Vfuse
+Text Label 1700 3550 3    50   ~ 0
+Vfuse
 $EndSCHEMATC
